File: Hardware/Control Hub.sch (EAGLE design)
At the start: 22 parts, among them IC1 LM555D, IC2 74AS08D, IC3 74AS08D

Commit message: Fixed board sizing and added logo
Added gitignore as well
Changed lines of the file:
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@@
 <pinref part="IC2" gate="P" pin="VCC"/>
 <pinref part="IC3" gate="P" pin="VCC"/>
+<junction x="91.44" y="10.16"/>
 </segment>
 </net>
@@
 <pinref part="IC2" gate="P" pin="GND"/>
 <pinref part="IC3" gate="P" pin="GND"/>
+<junction x="116.84" y="2.54"/>
 </segment>
 </net>
